Commit message: add the first link

File: scara_description/urdf/scara_arm.xacro (robot description, xacro)
@@ -3,5 +3,8 @@
     <xacro:property name="base_length" value="0.6"/>
     <xacro:property name="base_width" value="0.6"/>
-    <xacro:property name="base_height" value="0.1"/>
+    <xacro:property name="base_height" value="0.3"/>
+    <xacro:property name="link_length" value="0.6"/>
+    <xacro:property name="link_width" value="0.1"/>
+    <xacro:property name="link_height" value="0.05"/>
     <link name="base_footprint"/>
     <link name="base_link">
@@ -11,4 +14,13 @@
             </geometry>
             <origin xyz="0 0 0" rpy="0 0 0"/>
+            <material name="grey"/>
+        </visual>
+    </link>
+    <link name="link_1">
+        <visual>
+            <geometry>
+                <box size="${link_length} ${link_width} ${link_height}"/>
+            </geometry>
+            <origin xyz="${-link_length/2 + 0.03} 0 0" rpy="0 0 0"/>
             <material name="blue"/>
         </visual>
@@ -19,3 +31,11 @@
         <origin xyz="0 0 ${base_height/2}" rpy="0 0 0"/>
     </joint>
+    <joint name="base_joint_1" type="revolute">
+        <parent link="base_link"/>
+        <child link="link_1"/>
+        <origin xyz="${-link_length/2 + 0.03} 0 ${(base_height + link_height)/2}" rpy="0 0 0"/>
+        <axis xyz="0 0 1"/>
+        <limit lower="0" upper="${pi}" effort="100" velocity="100"/>
+        <dynamics friction="1000" damping="1000"/>
+    </joint>
 </robot>

Commit message: add second link

File: scara_description/urdf/scara_arm.xacro (robot description, xacro)
@@ -7,4 +7,7 @@
     <xacro:property name="link_width" value="0.1"/>
     <xacro:property name="link_height" value="0.05"/>
+    <xacro:property name="link_3_radius" value="0.1"/>
+    <xacro:property name="link_3_length" value="0.3"/>
+    <xacro:property name="offset" value="0.05"/>
     <link name="base_footprint"/>
     <link name="base_link">
@@ -22,6 +25,15 @@
                 <box size="${link_length} ${link_width} ${link_height}"/>
             </geometry>
-            <origin xyz="${-link_length/2 + 0.03} 0 0" rpy="0 0 0"/>
+            <origin xyz="${-link_length/2 + offset} 0 0" rpy="0 0 0"/>
             <material name="blue"/>
+        </visual>
+    </link>
+    <link name="link_2">
+        <visual>
+            <geometry>
+                <box size="${link_length} ${link_width} ${link_height}"/>
+            </geometry>
+            <origin xyz="${-link_length/2 + offset} 0 ${link_height/2}" rpy="0 0 0"/>
+            <material name="orange"/>
         </visual>
     </link>
@@ -31,10 +43,18 @@
         <origin xyz="0 0 ${base_height/2}" rpy="0 0 0"/>
     </joint>
-    <joint name="base_joint_1" type="revolute">
+    <joint name="joint_1" type="revolute">
         <parent link="base_link"/>
         <child link="link_1"/>
-        <origin xyz="${-link_length/2 + 0.03} 0 ${(base_height + link_height)/2}" rpy="0 0 0"/>
+        <origin xyz="${-link_length/2 + offset} 0 ${(base_height + link_height)/2}" rpy="0 0 0"/>
         <axis xyz="0 0 1"/>
-        <limit lower="0" upper="${pi}" effort="100" velocity="100"/>
+        <limit lower="${-pi/2}" upper="${pi/2}" effort="100" velocity="100"/>
+        <dynamics friction="1000" damping="1000"/>
+    </joint>
+    <joint name="joint_2" type="revolute">
+        <parent link="link_1"/>
+        <child link="link_2"/>
+        <origin xyz="${-link_length + offset} 0 ${link_height/2}" rpy="0 0 0"/>
+        <axis xyz="0 0 1"/>
+        <limit lower="${-pi/2}" upper="${pi/2}" effort="100" velocity="100"/>
         <dynamics friction="1000" damping="1000"/>
     </joint>

Commit message: add the third link

File: scara_description/urdf/scara_arm.xacro (robot description, xacro)
@@ -7,6 +7,6 @@
     <xacro:property name="link_width" value="0.1"/>
     <xacro:property name="link_height" value="0.05"/>
-    <xacro:property name="link_3_radius" value="0.1"/>
-    <xacro:property name="link_3_length" value="0.3"/>
+    <xacro:property name="link_3_radius" value="0.02"/>
+    <xacro:property name="link_3_length" value="0.4"/>
     <xacro:property name="offset" value="0.05"/>
     <link name="base_footprint"/>
@@ -35,4 +35,13 @@
             </geometry>
             <origin xyz="${-link_length/2 + offset} 0 ${link_height/2}" rpy="0 0 0"/>
+            <material name="blue"/>
+        </visual>
+    </link>
+    <link name="link_3">
+        <visual>
+            <geometry>
+                <cylinder radius="${link_3_radius}" length="${link_3_length}"/>
+            </geometry>
+            <origin xyz="0 0 ${-link_3_length/2}" rpy="0 0 0"/>
             <material name="orange"/>
         </visual>
@@ -59,3 +68,11 @@
         <dynamics friction="1000" damping="1000"/>
     </joint>
+    <joint name="joint_3" type="prismatic">
+        <parent link="link_2"/>
+        <child link="link_3"/>
+        <origin xyz="${-link_length + offset + link_3_radius*2} 0 0" rpy="0 0 0"/>
+        <axis xyz="0 0 1"/>
+        <limit lower="0" upper="1" effort="100" velocity="100"/>
+        <dynamics friction="1000" damping="1000"/>
+    </joint>
 </robot>

Commit message: add collision to link

File: scara_description/urdf/scara_arm.xacro (robot description, xacro)
@@ -19,4 +19,10 @@
             <material name="grey"/>
         </visual>
+        <collision>
+            <geometry>
+                <box size="${base_length} ${base_width} ${base_height}"/>
+            </geometry>
+            <origin xyz="0 0 0" rpy="0 0 0"/>
+        </collision>
     </link>
     <link name="link_1">
@@ -28,4 +34,10 @@
             <material name="blue"/>
         </visual>
+        <collision>
+            <geometry>
+                <box size="${link_length} ${link_width} ${link_height}"/>
+            </geometry>
+            <origin xyz="${-link_length/2 + offset} 0 0" rpy="0 0 0"/>
+        </collision>
     </link>
     <link name="link_2">
@@ -37,4 +49,10 @@
             <material name="blue"/>
         </visual>
+        <collision>
+            <geometry>
+                <box size="${link_length} ${link_width} ${link_height}"/>
+            </geometry>
+            <origin xyz="${-link_length/2 + offset} 0 ${link_height/2}" rpy="0 0 0"/>
+        </collision>
     </link>
     <link name="link_3">
@@ -46,4 +64,10 @@
             <material name="orange"/>
         </visual>
+        <collision>
+            <geometry>
+                <cylinder radius="${link_3_radius}" length="${link_3_length}"/>
+            </geometry>
+            <origin xyz="0 0 ${-link_3_length/2}" rpy="0 0 0"/>
+        </collision>
     </link>
     <joint name="base_joint" type="fixed">
