Commit message: add inertia macros

File: scara_description/urdf/common_properties.xacro (robot description, xacro)
@@ -10,3 +10,21 @@
         <color rgba="1 0.64 0 1"/>
     </material>
+    <xacro:macro name="box_inertia" params="m l w h xyz rpy">
+        <inertial>
+            <origin xyz="${xyz}" rpy="${rpy}"/>
+            <mass value="${m}" />
+            <inertia ixx="${(m/12) * (h*h + l*l)}" ixy="0" ixz="0"
+                     iyy="${(m/12) * (w*w + l*l)}" iyz="0"
+                     izz="${(m/12) * (w*w + h*h)}"/>
+        </inertial>
+    </xacro:macro>
+    <xacro:macro name="cylinder_inertia" params="m r l xyz rpy">
+        <inertial>
+            <origin xyz="${xyz}" rpy="${rpy}"/>
+            <mass value="${m}"/>
+            <inertia ixx="${(m/12)*(3*r*r + l*l)}" ixy="0" ixz="0"
+                     iyy="${(m/12)*(3*r*r + l*l)}" iyz="0"
+                     izz="${m*r*r/2.0}"/>
+        </inertial>
+    </xacro:macro>
 </robot>
