Commit message: add inertial to links

File: scara_description/urdf/scara.urdf.xacro (robot description, xacro)
@@ -1,5 +1,5 @@
 <?xml version="1.0"?>
 <robot name="scara" xmlns:xacro="http://www.ros.org/wiki/xacro">
+    <xacro:include filename="common_properties.xacro"/>
     <xacro:include filename="scara_arm.xacro"/>
-    <xacro:include filename="common_properties.xacro"/>
 </robot>

File: scara_description/urdf/scara_arm.xacro (robot description, xacro)
@@ -25,4 +25,6 @@
             <origin xyz="0 0 0" rpy="0 0 0"/>
         </collision>
+        <xacro:box_inertia m="50" l="${base_length * 2}" w="${base_width*2}" h="${base_height}"
+                            xyz="0 0 0" rpy="0 0 0"/>
     </link>
     <link name="link_1">
@@ -40,4 +42,6 @@
             <origin xyz="${-link_length/2 + offset} 0 0" rpy="0 0 0"/>
         </collision>
+        <xacro:box_inertia m="5" l="${2*link_length}" w="${2*base_width}" h="${base_height}"
+                            xyz="${-link_length/2 + offset} 0 0" rpy="0 0 0"/>
     </link>
     <link name="link_2">
@@ -55,4 +59,6 @@
             <origin xyz="${-link_length/2 + offset} 0 ${link_height/2}" rpy="0 0 0"/>
         </collision>
+        <xacro:box_inertia m="5" l="${2*link_length}" w="${2*base_width}" h="${base_height}"
+                            xyz="${-link_length/2 + offset} 0 ${link_height/2}" rpy="0 0 0"/>
     </link>
     <link name="link_3">
@@ -70,4 +76,6 @@
             <origin xyz="0 0 ${-link_3_length/2}" rpy="0 0 0"/>
         </collision>
+        <xacro:cylinder_inertia m="5" r="${2*link_3_radius}" l="${2*link_3_length}"
+                            xyz="0 0 ${-link_3_length/2}" rpy="0 0 0"/>
     </link>
     <joint name="base_joint" type="fixed">
@@ -97,5 +105,5 @@
         <origin xyz="${-link_length + offset + link_3_radius*2} 0 0" rpy="0 0 0"/>
         <axis xyz="0 0 1"/>
-        <limit lower="0" upper="1" effort="100" velocity="100"/>
+        <limit lower="0" upper="0.4" effort="100" velocity="100"/>
         <dynamics friction="1000" damping="1000"/>
     </joint>
